File: PCB_uitlezen_gsm/PCB_uitlezen_gsm.kicad_pcb (KiCad board)
At the start: 2 copper layers, 66.8 x 45 mm, 23 parts, among them J1 Conn_01x04_Pin, J2 Barrel_Jack, SW1 EN, SW2 FLASH, U1 ESP32-WROOM-32, U2 MP1584, U3 AMS1117-3.3

Commit message: update pcb uitlezen gsm design 2
Parts:
- SCHERM1, SCHERM2, SCHERM3: footprint Connector_PinHeader_2.00mm:PinHeader_1x09_P2.00mm_Vertical -> Connector_PinHeader_2.54mm:PinHeader_1x09_P2.54mm_Vertical
- moved SCHERM2 1.76 mm to (141.0, 111.8)
- moved SCHERM1 1.36 mm to (140.7, 107.4)
- moved SCHERM3 1.02 mm to (115.8, 111.8)
Routing:
- net +3.3V: track 215.0 -> 221.8 mm
- net GND: track 45.5 -> 38.9 mm, vias 22 -> 23
- net GPIO23: track 63.9 -> 68.2 mm
- net GPIO27: track 21.5 -> 23.9 mm
- net GPIO26: track 23.1 -> 25.2 mm
- net GPIO15: track 18.0 -> 16.0 mm
- net GPIO2: track 24.1 -> 22.6 mm
- net GPIO18: track 55.2 -> 56.6 mm
- net GPIO14: track 37.5 -> 38.7 mm
- net GPIO4: track 16.7 -> 15.9 mm
- net GPIO12: track 33.7 -> 33.1 mm
Other:
- board size 66.8 x 45 mm -> 69.8 x 46.7 mm

Commit message: update pcb design 2
Parts:
- C1: value 100uF/6.3V -> 47uF/6.3V
- J1: footprint Connector_PinHeader_2.00mm:PinHeader_1x04_P2.00mm_Vertical -> Connector_PinHeader_2.54mm:PinHeader_1x04_P2.54mm_Vertical
- moved J1 2.09 mm to (138.7, 86.6)
- moved J2 1.78 mm to (91.9, 104.4)
Routing:
- net +3.3V: track 221.8 -> 205.9 mm
- net TX0: track 17.6 -> 14.7 mm, vias 1 -> 2
- net GND: track 38.9 -> 37.2 mm, vias 23 -> 22
- net Net-(J2-Pad2): track 11.1 -> 10.4 mm
- net RX0: track 13.8 -> 14.4 mm
Other:
- board size 69.8 x 46.7 mm -> 65.8 x 46.7 mm
