File: pcb_morse/pcb_morse.kicad_pcb (KiCad board)
At the start: 2 copper layers, 65.5 x 61 mm, 41 parts, among them J2 Conn_01x04_Pin, Q1 BSS138, Q2 BSS138, Q3 MMBT3906, SW1 EN

Commit message: update pcb design 2
Parts:
- added SW2: FLASH, Button_Switch_SMD:SW_DIP_SPSTx01_Slide_Copal_CHS-01B_W7.62mm_P1.27mm, F.Cu at (80.8, 40.6)
- J2, ULTRASONIC-SENSOR1: footprint Connector_PinHeader_2.00mm:PinHeader_1x04_P2.00mm_Vertical -> Connector_PinHeader_2.54mm:PinHeader_1x04_P2.54mm_Vertical
- moved ULTRASONIC-SENSOR1 2.11 mm to (89.9, 70.1)
- moved LED1 1.52 mm to (90.4, 53.1)
Routing:
- net Net-(LED1-A): track 11.6 -> 24.8 mm
- net GPIO17-5V: track 11.7 -> 13.0 mm
- net TX0: track 29.6 -> 30.7 mm
- net VDD: track 81.4 -> 81.9 mm

Commit message: clean up
Parts:
- removed R10: 1k, Resistor_SMD:R_0805_2012Metric_Pad1.20x1.40mm_HandSolder
- added U1: EL817, Package_DIP:DIP-4_W7.62mm, F.Cu at (50.3, 64.0)
- C1: value 100uF/6.3V -> 47uF/6.3V
- D1: value D -> 1n4148
- Q3: value MMBT3906 -> Q_NPN_BCE
- moved Kroonsteen1 17.1 mm to (78.0, 84.3)
- moved R9 14.0 mm to (59.9, 65.5)
- moved Q3 13.5 mm to (63.3, 65.8)
- moved Relais1 7.07 mm to (55.3, 69.7)
- moved R8 0.52 mm to (52.1, 53.8)
- moved D1 0.11 mm to (66.0, 60.7)
Connections:
- D1 pad 1: Net-(D1-K) -> VDD
- D1 pad 2: GND -> Net-(D1-A)
- Kroonsteen1 pad 3: Net-(Kroonsteen1-Pin_3) -> GND
- Q3 pad 2: +12V -> Net-(D1-A)
- Q3 pad 3: Net-(D1-K) -> GND
- R8 pad 1: Net-(Q3-B) -> VDD
- R8 pad 2: GPIO32 -> Net-(R8-Pad2)
- R9 pad 1: +12V -> Net-(R9-Pad1)
- R9 pad 2: GND -> Net-(Q3-B)
- Relais1 pad 1: Net-(Kroonsteen1-Pin_3) -> +12V
- Relais1 pad 2: GND -> Net-(D1-A)
- Relais1 pad 5: Net-(D1-K) -> VDD
Routing:
- net Net-(Kroonsteen1-Pin_3): track 29.9 -> 0.00 mm
- net Net-(D1-A): track 0.00 -> 24.0 mm
- net VDD: track 81.9 -> 105.2 mm
- net Net-(D1-K): track 21.4 -> 0.00 mm
- net Net-(Kroonsteen1-Pin_2): track 12.1 -> 25.4 mm
- net Net-(R8-Pad2): track 0.00 -> 11.3 mm
- net Net-(R9-Pad1): track 0.00 -> 11.1 mm, vias 0 -> 1
- net GPIO32: track 7.00 -> 16.6 mm
- net Net-(Kroonsteen1-Pin_1): track 9.92 -> 18.1 mm
- net +12V: track 29.2 -> 21.2 mm
- net GND: vias 30 -> 28
Other:
- board text added: "COM"
