File: pcb_morse/pcb_morse.kicad_sch (KiCad schematic)
At the start: 42 parts, among them J1 Conn_01x04_Pin, J2 Barrel_Jack, Q1 BSS138, Q2 BSS138, Q3 MMBT3906, SW1 EN, SW2 FLASH, U1 ESP32-WROOM-32, U2 MP1584, U3 AMS1117-3.3

Commit message: update pcb design 2
Parts:
- removed SW2: FLASH, Button_Switch_SMD:SW_DIP_SPSTx01_Slide_Copal_CHS-01B_W7.62mm_P1.27mm, symbol Switch:SW_Push
- added SW1: FLASH, Button_Switch_SMD:SW_DIP_SPSTx01_Slide_Copal_CHS-01B_W7.62mm_P1.27mm, symbol Switch:SW_Push
- J1, ULTRASONIC-SENSOR1: footprint Connector_PinHeader_2.00mm:PinHeader_1x04_P2.00mm_Vertical -> Connector_PinHeader_2.54mm:PinHeader_1x04_P2.54mm_Vertical
Connections:
- net GND: now also SW1.2
- net GPIO0: now also SW1.1
Changed lines of the file:
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@@
   (junction (at 163.83 78.74) (diameter 0) (color 0 0 0 0)
+  )
+  (junction (at 111.76 33.02) (diameter 0) (color 0 0 0 0)
   )
   (junction (at 120.65 175.26) (diameter 0) (color 0 0 0 0)
@@
     (stroke (width 0) (type default))
   )
+  (wire (pts (xy 128.27 33.02) (xy 132.08 33.02))
+    (stroke (width 0) (type default))
+  )
   (wire (pts (xy 40.64 151.13) (xy 40.64 153.67))
     (stroke (width 0) (type default))
@@
     (stroke (width 0) (type default))
   )
+  (wire (pts (xy 111.76 33.02) (xy 118.11 33.02))
+    (stroke (width 0) (type default))
+  )
   (wire (pts (xy 107.95 52.07) (xy 111.76 52.07))
     (stroke (width 0) (type default))
@@
     (stroke (width 0) (type default))
   )
-  (wire (pts (xy 107.95 33.02) (xy 115.57 33.02))
+  (wire (pts (xy 107.95 33.02) (xy 111.76 33.02))
     (stroke (width 0) (type default))
   )
@@
     (stroke (width 0) (type default))
   )
+  (wire (pts (xy 111.76 31.75) (xy 111.76 33.02))
+    (stroke (width 0) (type default))
+  )
   (wire (pts (xy 222.25 26.67) (xy 218.44 26.67))
     (stroke (width 0) (type default))
@@
   )
   (wire (pts (xy 163.83 83.82) (xy 163.83 85.09))
-    (stroke (width 0) (type default))
-  )
-  (wire (pts (xy 125.73 33.02) (xy 132.08 33.02))
     (stroke (width 0) (type default))
   )
@@
     )
   )
-  (global_label "GPIO0" (shape input) (at 111.76 33.02 90) (fields_autoplaced)
+  (global_label "GPIO0" (shape input) (at 111.76 31.75 90) (fields_autoplaced)
     (effects (font (size 1.27 1.27)) (justify left))
-    (property "Intersheetrefs" "${INTERSHEET_REFS}" (at 111.76 24.4294 90)
+    (property "Intersheetrefs" "${INTERSHEET_REFS}" (at 111.76 23.1594 90)
       (effects (font (size 1.27 1.27)) (justify left) hide)
     )
@@
       (effects (font (size 1.27 1.27)) (justify left))
     )
-    (property "Footprint" "Connector_PinHeader_2.00mm:PinHeader_1x04_P2.00mm_Vertical" (at 198.12 119.38 0)
+    (property "Footprint" "Connector_PinHeader_2.54mm:PinHeader_1x04_P2.54mm_Vertical" (at 198.12 119.38 0)
       (effects (font (size 1.27 1.27)) hide)
     )
@@
       (effects (font (size 1.27 1.27)))
     )
-    (property "Footprint" "Connector_PinHeader_2.00mm:PinHeader_1x04_P2.00mm_Vertical" (at 213.36 29.21 0)
+    (property "Footprint" "Connector_PinHeader_2.54mm:PinHeader_1x04_P2.54mm_Vertical" (at 213.36 29.21 0)
       (effects (font (size 1.27 1.27)) hide)
     )
@@
     )
   )
-  (symbol (lib_name "SW_Push_1") (lib_id "Switch:SW_Push") (at 120.65 33.02 0) (unit 1)
-    (in_bom yes) (on_board yes) (dnp no) (fields_autoplaced)
-    (property "Reference" "SW2" (at 120.65 26.67 0)
-      (effects (font (size 1.27 1.27)))
-    )
-    (property "Value" "FLASH" (at 120.65 29.21 0)
-      (effects (font (size 1.27 1.27)))
-    )
-    (property "Footprint" "Button_Switch_SMD:SW_DIP_SPSTx01_Slide_Copal_CHS-01B_W7.62mm_P1.27mm" (at 120.65 27.94 0)
-      (effects (font (size 1.27 1.27)) hide)
-    )
-    (property "Datasheet" "~" (at 120.65 27.94 0)
-      (effects (font (size 1.27 1.27)) hide)
-    )
-    (pin "1")
-    (pin "1")
-    (instances
-      (project "esp32_pcb"
-        (path "/1568d5f0-bcdb-494d-bbf5-b93d65138b4f"
-          (reference "SW2") (unit 1)
-        )
-      )
-      (project "pcb_morse"
-        (path "/a7bc0285-62e4-4eee-a4a4-109b456cc260"
-          (reference "SW3") (unit 1)
-        )
-      )
-    )
-  )
   (symbol (lib_id "Device:R") (at 106.68 73.66 90) (unit 1)
     (in_bom yes) (on_board yes) (dnp no) (fields_autoplaced)
@@
         )
       )
+    )
+  )
+  (symbol (lib_name "SW_Push_2") (lib_id "Switch:SW_Push") (at 123.19 33.02 0) (unit 1)
+    (in_bom yes) (on_board yes) (dnp no) (fields_autoplaced)
+    (property "Reference" "SW1" (at 123.19 26.67 0)
+      (effects (font (size 1.27 1.27)))
+    )
+    (property "Value" "FLASH" (at 123.19 29.21 0)
+      (effects (font (size 1.27 1.27)))
+    )
+    (property "Footprint" "Button_Switch_SMD:SW_DIP_SPSTx01_Slide_Copal_CHS-01B_W7.62mm_P1.27mm" (at 123.19 27.94 0)
+      (effects (font (size 1.27 1.27)) hide)
+    )
+    (property "Datasheet" "~" (at 123.19 27.94 0)
+      (effects (font (size 1.27 1.27)) hide)
+    )
+    (pin "1")
+    (pin "2")
+    (instances
+      (project "esp32_pcb"
+        (path "/1568d5f0-bcdb-494d-bbf5-b93d65138b4f"
+          (reference "SW1") (unit 1)
+        )
+      )
+      (project "pcb_morse"
+        (path "/a7bc0285-62e4-4eee-a4a4-109b456cc260"
+          (reference "SW2") (unit 1)
+        )
+      )

Commit message: clean up
Parts:
- removed Q3: MMBT3906, Package_TO_SOT_SMD:SOT-23, symbol Transistor_BJT:MMBT3906
- removed R10: 1k, Resistor_SMD:R_0805_2012Metric_Pad1.20x1.40mm_HandSolder, symbol Device:R
- added Q3: Q_NPN_BCE, Package_TO_SOT_SMD:SOT-23, symbol Device:Q_NPN_BCE
- added U1: EL817, Package_DIP:DIP-4_W7.62mm, symbol Isolator:EL817
- C1: value 100uF/6.3V -> 47uF/6.3V
- D1: value D -> 1n4148
Connections:
- net +12V: now also Relais1.1; no longer R9.1
- net GND: now also Kroonsteen1.3 (Pin_3), Q3.3 (E); no longer D1.2 (A), R9.2, Relais1.2
- net GPIO32: now also U1.2; no longer R8.2
- net VDD: now also D1.1 (K), R8.1, Relais1.5, U1.4
- new net: R9.1, U1.3
- new net: Q3.1 (B), R9.2
- new net: D1.2 (A), Q3.2 (C), Relais1.2
- new net: R8.2, U1.1
Other:
- moved on the sheet: Kroonsteen1, Relais1
